Commit message: added camera macro

File: src/slam/urdf/lidar.xacro (robot description, xacro)
@@ -57,3 +57,57 @@
         </gazebo>
     </xacro:macro>
+	<xacro:macro name="camera" params="namespace">
+        <!-- Camera Link -->
+        <link name="${namespace}/camera_frame">
+            <visual>
+                <geometry>
+                    <box size="0.03 0.08 0.03"/>
+                </geometry>
+                <material name="black"/>
+            </visual>
+            <collision>
+                <geometry>
+                    <box size="0.03 0.08 0.03"/>
+                </geometry>
+            </collision>
+            <inertial>
+                <mass value="0.1"/>
+                <origin xyz="0 0 0"/>
+                <inertia ixx="0.000083" ixy="0" ixz="0"
+                         iyy="0.000083" iyz="0"
+                         izz="0.000083"/>
+            </inertial>
+        </link>
+        <!-- Camera Joint -->
+        <joint name="${namespace}/camera_joint" type="fixed">
+            <parent link="${namespace}/base_link"/>
+            <child link="${namespace}/camera_frame"/>
+            <origin xyz="0.15 0 0.05" rpy="0 0 0"/>
+        </joint>
+        <!-- Gazebo Plugin Configuration -->
+        <gazebo reference="${namespace}/camera_frame">
+            <sensor name="${namespace}_camera" type="camera">
+                <update_rate>30.0</update_rate>
+                <camera>
+                    <horizontal_fov>1.3962634</horizontal_fov>
+                    <image>
+                        <width>640</width>
+                        <height>480</height>
+                        <format>R8G8B8</format>
+                    </image>
+                    <clip>
+                        <near>0.02</near>
+                        <far>300</far>
+                    </clip>
+                </camera>
+                <plugin name="${namespace}_camera_controller" filename="libgazebo_ros_camera.so">
+                    <ros>
+                        <remapping>image_raw:=/${namespace}/image_raw</remapping>
+                        <remapping>camera_info:=/${namespace}/camera_info</remapping>
+                    </ros>
+                    <frame_name>${namespace}/camera_frame</frame_name>
+                </plugin>
+            </sensor>
+        </gazebo>
+    </xacro:macro>
 </robot>
